File: HW/pcb_heater_element.kicad_pcb (KiCad board)
At the start: 2 copper layers, 130.2 x 300 mm, 0 parts

Commit message: QOL changes on pcb, fixed wrong ACDC brick polarity xD
Other:
- board size 130.2 x 300 mm -> 107.2 x 300 mm
- board text removed: "JLCJLCJLC"
Changed lines of the file:
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@@
     )
     (pad_to_mask_clearance 0)
-    (grid_origin 121.250001 72)
+    (grid_origin 176.750001 57)
     (pcbplotparams
       (layerselection 0x00010fc_ffffffff)
@@
       (xy 208.75 344)
     ) (layer "Dwgs.User") (width 0.15) (fill none))
-  (gr_rect (start 215.750001 65) (end 221.750001 59) (layer "Dwgs.User") (width 0.15) (fill none))
   (gr_rect (start 208.75 59) (end 202.75 65) (layer "Dwgs.User") (width 0.15) (fill none))
   (gr_rect (start 114.75 344) (end 120.75 350) (layer "Dwgs.User") (width 0.15) (fill none))
@@
   (gr_line (start 114.750011 324) (end 208.750011 324) (layer "Dwgs.User") (width 0.15))
   (gr_line (start 114.750004 170) (end 208.750004 170) (layer "Dwgs.User") (width 0.15))
-  (gr_rect (start 227.750001 65) (end 233.750001 59) (layer "Dwgs.User") (width 0.15) (fill none))
   (gr_rect (start 114.75 59) (end 120.75 65) (layer "Dwgs.User") (width 0.15) (fill none))
   (gr_line (start 114.750006 214) (end 208.750006 214) (layer "Dwgs.User") (width 0.15))
@@
   (gr_arc (start 111.157701 216.269136) (mid 111.6577 215.769137) (end 112.157698 216.269136) (layer "Edge.Cuts") (width 0.1))
   (gr_line (start 111.75 223.84) (end 111.75 355.5) (layer "Edge.Cuts") (width 0.1))
+  (gr_line (start 177.542894 357) (end 210.25 357) (layer "Edge.Cuts") (width 0.1))
+  (gr_line (start 176.042894 355.499999) (end 148.042895 355.499998) (layer "Edge.Cuts") (width 0.1))
   (gr_line (start 211.75 214.5) (end 211.75 58.5) (layer "Edge.Cuts") (width 0.1))
-  (gr_line (start 210.25 357) (end 113.25 357) (layer "Edge.Cuts") (width 0.1))
+  (gr_circle (center 206.250001 319.5) (end 210.350001 319.5) (layer "Edge.Cuts") (width 0.1) (fill none))
+  (gr_line (start 146.542895 356.999997) (end 113.25 357) (layer "Edge.Cuts") (width 0.1))
   (gr_line (start 112.1577 222.269138) (end 112.157698 216.269136) (layer "Edge.Cuts") (width 0.1))
-  (gr_line (start 113.25 57) (end 210.25 57) (layer "Edge.Cuts") (width 0.1))
+  (gr_line (start 113.25 57) (end 146.250002 56.999998) (layer "Edge.Cuts") (width 0.1))
   (gr_arc (start 205.675 220.9) (mid 204.501525 219.288514) (end 205.6 217.625) (layer "Edge.Cuts") (width 0.1))
   (gr_line (start 105.75 220.9) (end 111.230732 223.27811) (layer "Edge.Cuts") (width 0.1))
   (gr_arc (start 113.25 357) (mid 112.18934 356.56066) (end 111.75 355.5) (layer "Edge.Cuts") (width 0.1))
+  (gr_arc (start 176.750001 57.5) (mid 176.896448 57.146447) (end 177.250001 57) (layer "Edge.Cuts") (width 0.1))
   (gr_arc (start 111.750732 214.5) (mid 111.657701 214.869137) (end 111.400732 215.15) (layer "Edge.Cuts") (width 0.1))
+  (gr_arc (start 147.042894 356.499998) (mid 147.335787 355.79289) (end 148.042895 355.499998) (layer "Edge.Cuts") (width 0.1))
   (gr_arc (start 112.1577 222.269138) (mid 111.657701 222.769137) (end 111.157702 222.269138) (layer "Edge.Cuts") (width 0.1))
   (gr_line (start 111.157701 216.269136) (end 111.157702 222.269138) (layer "Edge.Cuts") (width 0.1))
   (gr_line (start 111.400732 215.15) (end 105.675 217.625) (layer "Edge.Cuts") (width 0.1))
+  (gr_arc (start 176.750001 57.5) (mid 176.457108 58.207107) (end 175.750001 58.5) (layer "Edge.Cuts") (width 0.1))
   (gr_arc (start 210.25 57) (mid 211.31066 57.43934) (end 211.75 58.5) (layer "Edge.Cuts") (width 0.1))
   (gr_line (start 211.749268 223.84) (end 211.75 355.5) (layer "Edge.Cuts") (width 0.1))
   (gr_line (start 111.750732 214.5) (end 111.75 58.5) (layer "Edge.Cuts") (width 0.1))
   (gr_arc (start 211.75 355.5) (mid 211.31066 356.56066) (end 210.25 357) (layer "Edge.Cuts") (width 0.1))
+  (gr_arc (start 177.542894 357) (mid 177.18934 356.853553) (end 177.042893 356.5) (layer "Edge.Cuts") (width 0.1))
+  (gr_line (start 147.750002 58.499999) (end 175.750001 58.5) (layer "Edge.Cuts") (width 0.1))
   (gr_line (start 211.4 215.15) (end 205.6 217.625) (layer "Edge.Cuts") (width 0.1))
   (gr_arc (start 105.75 220.9) (mid 104.576521 219.288528) (end 105.675 217.625) (layer "Edge.Cuts") (width 0.1))
   (gr_arc (start 211.75 214.5) (mid 211.656969 214.869137) (end 211.4 215.15) (layer "Edge.Cuts") (width 0.1))
   (gr_arc (start 211.23 223.27811) (mid 211.565616 223.488836) (end 211.749268 223.84) (layer "Edge.Cuts") (width 0.1))
+  (gr_arc (start 146.250002 56.999998) (mid 146.603556 57.146445) (end 146.750003 57.499998) (layer "Edge.Cuts") (width 0.1))
+  (gr_arc (start 176.042894 355.499999) (mid 176.750001 355.792892) (end 177.042894 356.499999) (layer "Edge.Cuts") (width 0.1))
   (gr_line (start 205.675 220.9) (end 211.23 223.27811) (layer "Edge.Cuts") (width 0.1))
-  (gr_rect (start 214.750001 58) (end 234.750001 66) (layer "Edge.Cuts") (width 0.1) (fill none))
+  (gr_circle (center 117.250001 88.5) (end 121.350001 88.5) (layer "Edge.Cuts") (width 0.1) (fill none))
+  (gr_line (start 210.250002 57) (end 177.250001 57) (layer "Edge.Cuts") (width 0.1))
   (gr_arc (start 111.230732 223.27811) (mid 111.566348 223.488836) (end 111.75 223.84) (layer "Edge.Cuts") (width 0.1))
+  (gr_arc (start 147.042894 356.499998) (mid 146.896447 356.85355) (end 146.542895 356.999997) (layer "Edge.Cuts") (width 0.1))
   (gr_arc (start 111.75 58.5) (mid 112.18934 57.43934) (end 113.25 57) (layer "Edge.Cuts") (width 0.1))
-  (gr_text "JLCJLCJLC" (at 224.750001 62) (layer "B.SilkS")
-    (effects (font (size 1 1) (thickness 0.15)) (justify mirror))
-  )
+  (gr_arc (start 147.750002 58.499999) (mid 147.042895 58.207106) (end 146.750002 57.499999) (layer "Edge.Cuts") (width 0.1))
   (gr_text "JLCJLCJLCJLC" (at 161.750001 352.5) (layer "F.SilkS")
     (effects (font (size 1 1) (thickness 0.25)))
@@
     (polygon
       (pts
-        (xy 234.000001 65.25)
-        (xy 215.500001 65.25)
-        (xy 215.500001 58.75)
-        (xy 234.000001 58.75)
-      )
-    )
-  )
-  (zone (net 0) (net_name "") (layer "F.Cu") (hatch edge 0.508)
-    (connect_pads (clearance 0))
-    (min_thickness 0.254) (filled_areas_thickness no)
-    (fill yes (thermal_gap 0.508) (thermal_bridge_width 0.508))
-    (polygon
-      (pts
         (xy 208.75 344)
         (xy 208.749999 350)
@@
     (polygon
       (pts
-        (xy 221.750001 65)
-        (xy 215.750001 65)
-        (xy 215.750001 59)
-        (xy 221.750001 59)
-      )
-    )
-  )
-  (zone (net 0) (net_name "") (layer "F.Mask") (hatch edge 0.508)
-    (connect_pads (clearance 0))
-    (min_thickness 0.254) (filled_areas_thickness no)
-    (fill yes (thermal_gap 0.508) (thermal_bridge_width 0.508))
-    (polygon
-      (pts
         (xy 120.75 65)
         (xy 114.75 65)
@@
       )
     )
-  )
-  (zone (net 0) (net_name "") (layer "F.Mask") (hatch edge 0.508)
-    (connect_pads (clearance 0))
-    (min_thickness 0.254) (filled_areas_thickness no)
-    (fill yes (thermal_gap 0.508) (thermal_bridge_width 0.508))
-    (polygon
-      (pts
-        (xy 233.750001 65)
-        (xy 227.750001 65)
-        (xy 227.750001 59)
-        (xy 233.750001 59)
-      )
-    )

Commit message: revision 0
Other:
- board size 107.2 x 300 mm -> 107 x 300 mm
- board text added: "- trace width 1.5 mm - unit length = (2 lines + 2 arcs) = 81 * 2 + 17.27875 * 2 = 196.6 mm - total full units = 12 - first unit is 83.5 + 81 + (17.27875*2) = 199 mm - last unit is 83 mm - total trace length per heater: 2.64 m - total trace length (x3 heaters) ~= 7.9 m - track resistance at 20°C ~= 2.5 Ohm"
- board text removed: "- trace width 1.5 mm - unit length = (2 lines + 2 arcs) = 81 * 2 + 17.27875 * 2 = 196.6 mm - total full units = 12 - first unit is 83.5 + 81 + (17.27875*2) = 199 mm - last unit is 83 mm - total trace length per heater: 2.64 m - total trace length (x3 heaters) ~= 7.9 m"
