File: HW/pcb_heater_element.kicad_pcb (KiCad board)
At the start: 2 copper layers, 107 x 300 mm, 0 parts

Commit message: Readme and board fixes
Other:
- outline, holes or cut-outs redrawn
Changed lines of the file:
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@@
   (gr_rect (start 208.75 344) (end 202.75 350) (layer "Dwgs.User") (width 0.15) (fill none))
   (gr_line (start 114.750009 280) (end 208.750009 280) (layer "Dwgs.User") (width 0.15))
-  (gr_arc (start 111.157701 216.269136) (mid 111.6577 215.769137) (end 112.157698 216.269136) (layer "Edge.Cuts") (width 0.1))
   (gr_line (start 111.75 223.84) (end 111.75 355.5) (layer "Edge.Cuts") (width 0.1))
   (gr_line (start 181.750001 355.499997) (end 141.750001 355.499999) (layer "Edge.Cuts") (width 0.1))
   (gr_line (start 211.75 214.5) (end 211.75 58.5) (layer "Edge.Cuts") (width 0.1))
   (gr_circle (center 206.250001 319.5) (end 210.400001 319.5) (layer "Edge.Cuts") (width 0.1) (fill none))
-  (gr_line (start 112.1577 222.269138) (end 112.157698 216.269136) (layer "Edge.Cuts") (width 0.1))
   (gr_line (start 113.25 57) (end 140.250001 56.999999) (layer "Edge.Cuts") (width 0.1))
   (gr_arc (start 205.675 220.9) (mid 204.501525 219.288514) (end 205.6 217.625) (layer "Edge.Cuts") (width 0.1))
@@
   (gr_line (start 181.750001 58.499998) (end 141.750001 58.5) (layer "Edge.Cuts") (width 0.1))
   (gr_line (start 183.250001 356.999998) (end 210.25 357) (layer "Edge.Cuts") (width 0.1))
-  (gr_arc (start 112.1577 222.269138) (mid 111.657701 222.769137) (end 111.157702 222.269138) (layer "Edge.Cuts") (width 0.1))
   (gr_line (start 113.25 357) (end 140.250001 356.999999) (layer "Edge.Cuts") (width 0.1))
-  (gr_line (start 111.157701 216.269136) (end 111.157702 222.269138) (layer "Edge.Cuts") (width 0.1))
   (gr_line (start 111.400732 215.15) (end 105.84848 217.625) (layer "Edge.Cuts") (width 0.1))
   (gr_arc (start 182.750001 57.499998) (mid 182.457108 58.207105) (end 181.750001 58.499998) (layer "Edge.Cuts") (width 0.1))
