File: HW/pcb_heater_joiner.kicad_pcb (KiCad board)
At the start: 2 copper layers, 20 x 8 mm, 0 parts

Commit message: revision 0
Other:
- board text added: "JLCJLCJLCJLC"
- board text removed: "JLCJLCJLC"
Changed lines of the file:
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@@
       (sketchpadsonfab false)
       (subtractmaskfromsilk false)
-      (outputformat 3)
+      (outputformat 1)
       (mirror false)
       (drillshape 0)
@@
   (gr_rect (start 104.25 67.5) (end 110.25 61.5) (layer "Dwgs.User") (width 0.15) (fill none))
   (gr_rect (start 91.25 60.5) (end 111.25 68.5) (layer "Edge.Cuts") (width 0.1) (fill none))
-  (gr_text "JLCJLCJLC" (at 101.25 64.5) (layer "B.SilkS")
+  (gr_text "JLCJLCJLCJLC" (at 101.25 64.5) (layer "B.SilkS")
     (effects (font (size 1 1) (thickness 0.15)) (justify mirror))
   )
